Commit message: gazebo can't launch

File: src/basic_robot/description/gazebo_test.xacro (robot description, xacro)
@@ -1,4 +1,4 @@
 <?xml version="1.0" ?>
-<robot name="test" xmlns:xacro="http://www.ros.org/wiki/xacro">
+<robot name="my_bot" xmlns:xacro="http://www.ros.org/wiki/xacro">
   <link name="base_link">
   </link>
@@ -10,6 +10,6 @@
     <inertial>
       <origin xyz="0.0 0.0 0.0" rpy="0 0 0"/>
-      <mass value="0"/>
-      <inertia ixx="0.0" iyy="0.0" izz="0.0" ixy="0.0" iyz="0.0" ixz="0.0"/>
+      <mass value="10"/>
+      <inertia  ixx="0.41666666666666663" ixy="0" ixz="0" iyy="1.0416666666666665" iyz="0" izz="1.0416666666666665" />
     </inertial>
     <visual>
@@ -29,6 +29,6 @@
     <inertial>
       <origin xyz="0 0 0" rpy="0 0 0"/>
-      <mass value="0"/>
-      <inertia ixx="0.0" iyy="0.0" izz="0.0" ixy="-0.0" iyz="-0.0" ixz="0.0"/>
+      <mass value="5"/>
+      <inertia  ixx="0.5327296181012307" ixy="0" ixz="0" iyy="0.3035629514345639" iyz="0" izz="0.30416666666666675" />
     </inertial>
     <visual>
@@ -48,6 +48,6 @@
     <inertial>
       <origin xyz="0 0 0" rpy="0 0 0"/>
-      <mass value="0"/>
-      <inertia ixx="0.0" iyy="0.0" izz="0.0" ixy="-0.0" iyz="-0.0" ixz="0.0"/>
+      <mass value="5"/>
+      <inertia  ixx="0.5327295545949559" ixy="0" ixz="0" iyy="0.3035628879282892" iyz="0" izz="0.30416666666666675" />
     </inertial>
     <visual>

Commit message: gazebo shows - use file:// for stls

File: src/basic_robot/description/gazebo_test.xacro (robot description, xacro)
@@ -2,19 +2,16 @@
 <robot name="my_bot" xmlns:xacro="http://www.ros.org/wiki/xacro">
   <link name="base_link">
+    <origin xyz="0.0 0.0 0.0" rpy="0.0 0.0 0.0"/>
   </link>
   <joint name="base_joint" type="fixed">
     <parent link="base_link"/>
     <child link="chassis"/>
+    <origin xyz="0 0 0" rpy="0 0 0"/>
   </joint>
   <link name="chassis">
-    <inertial>
-      <origin xyz="0.0 0.0 0.0" rpy="0 0 0"/>
-      <mass value="10"/>
-      <inertia  ixx="0.41666666666666663" ixy="0" ixz="0" iyy="1.0416666666666665" iyz="0" izz="1.0416666666666665" />
-    </inertial>
     <visual>
       <origin xyz="0 0 0" rpy="0 0 0"/>
       <geometry>
-        <mesh filename="package://basic_robot/meshes/chassis.stl" scale="0.1 0.1 0.1"/>
+        <mesh filename="file://$(find basic_robot)/meshes/chassis.stl" scale="0.01 0.01 0.01"/>
       </geometry>
     </visual>
@@ -22,7 +19,12 @@
       <origin xyz="0 0 0" rpy="0 0 0"/>
       <geometry>
-        <mesh filename="package://basic_robot/meshes/chassis.stl" scale="0.1 0.1 0.1"/>
+        <mesh filename="file://$(find basic_robot)/meshes/chassis.stl" scale="0.01 0.01 0.01"/>
       </geometry>
     </collision>
+    <inertial>
+      <origin xyz="0.0 0.0 0.0" rpy="0 0 0"/>
+      <mass value="10"/>
+      <inertia  ixx="0.42" ixy="0" ixz="0" iyy="1.042" iyz="0" izz="1.042" />
+    </inertial>
   </link>
   <link name="left_wheel_1">
@@ -35,5 +37,5 @@
       <origin xyz="0.5 -0.0 -0.25" rpy="0 0 0"/>
       <geometry>
-        <mesh filename="package://basic_robot/meshes/left_wheel_1.stl" scale="0.1 0.1 0.1"/>
+        <mesh filename="file://$(find basic_robot)/meshes/left_wheel_1.stl" scale="0.01 0.01 0.01"/>
       </geometry>
     </visual>
@@ -41,5 +43,5 @@
       <origin xyz="0.5 -0.0 -0.25" rpy="0 0 0"/>
       <geometry>
-        <mesh filename="package://basic_robot/meshes/left_wheel_1.stl" scale="0.1 0.1 0.1"/>
+        <mesh filename="file://$(find basic_robot)/meshes/left_wheel_1.stl" scale="0.01 0.01 0.01"/>
       </geometry>
     </collision>
@@ -54,5 +56,5 @@
       <origin xyz="-0.5 -0.0 -0.25" rpy="0 0 0"/>
       <geometry>
-        <mesh filename="package://basic_robot/meshes/right_wheel_1.stl" scale="0.1 0.1 0.1"/>
+        <mesh filename="file://$(find basic_robot)/meshes/right_wheel_1.stl" scale="0.01 0.01 0.01"/>
       </geometry>
     </visual>
@@ -60,5 +62,5 @@
       <origin xyz="-0.5 -0.0 -0.25" rpy="0 0 0"/>
       <geometry>
-        <mesh filename="package://basic_robot/meshes/right_wheel_1.stl" scale="0.1 0.1 0.1"/>
+        <mesh filename="file://$(find basic_robot)/meshes/right_wheel_1.stl" scale="0.01 0.01 0.01"/>
       </geometry>
     </collision>
