Commit message: controller_manager fails to spawn

File: src/basic_robot/description/gazebo.xacro (robot description, xacro)
@@ -13,5 +13,5 @@
       <origin xyz="0 0 0" rpy="0 0 0"/>
       <geometry>
-        <mesh filename="file://$(find basic_robot)/meshes/chassis.stl" scale="0.01 0.01 0.01"/>
+        <mesh filename="file://$(find basic_robot)/meshes/chassis.stl" scale="0.1 0.1 0.1"/>
       </geometry>
     </visual>
@@ -19,5 +19,5 @@
       <origin xyz="0 0 0" rpy="0 0 0"/>
       <geometry>
-        <mesh filename="file://$(find basic_robot)/meshes/chassis.stl" scale="0.01 0.01 0.01"/>
+        <mesh filename="file://$(find basic_robot)/meshes/chassis.stl" scale="0.1 0.1 0.1"/>
       </geometry>
     </collision>
@@ -37,5 +37,5 @@
       <origin xyz="0.5 -0.0 -0.25" rpy="0 0 0"/>
       <geometry>
-        <mesh filename="file://$(find basic_robot)/meshes/left_wheel_1.stl" scale="0.01 0.01 0.01"/>
+        <mesh filename="file://$(find basic_robot)/meshes/left_wheel_1.stl" scale="0.1 0.1 0.1"/>
       </geometry>
     </visual>
@@ -43,5 +43,5 @@
       <origin xyz="0.5 -0.0 -0.25" rpy="0 0 0"/>
       <geometry>
-        <mesh filename="file://$(find basic_robot)/meshes/left_wheel_1.stl" scale="0.01 0.01 0.01"/>
+        <mesh filename="file://$(find basic_robot)/meshes/left_wheel_1.stl" scale="0.1 0.1 0.1"/>
       </geometry>
     </collision>
@@ -56,5 +56,5 @@
       <origin xyz="-0.5 -0.0 -0.25" rpy="0 0 0"/>
       <geometry>
-        <mesh filename="file://$(find basic_robot)/meshes/right_wheel_1.stl" scale="0.01 0.01 0.01"/>
+        <mesh filename="file://$(find basic_robot)/meshes/right_wheel_1.stl" scale="0.1 0.1 0.1"/>
       </geometry>
     </visual>
@@ -62,19 +62,27 @@
       <origin xyz="-0.5 -0.0 -0.25" rpy="0 0 0"/>
       <geometry>
-        <mesh filename="file://$(find basic_robot)/meshes/right_wheel_1.stl" scale="0.01 0.01 0.01"/>
+        <mesh filename="file://$(find basic_robot)/meshes/right_wheel_1.stl" scale="0.1 0.1 0.1"/>
       </geometry>
     </collision>
   </link>
-  <joint name="Revolute 1" type="continuous">
+  <joint name="Revolute1" type="continuous">
     <origin xyz="-0.5 0.0 0.25" rpy="0 0 0"/>
-    <parent link="base_link"/>
+    <parent link="chassis"/>
     <child link="left_wheel_1"/>
     <axis xyz="-1.0 0.0 0.0"/>
   </joint>
-  <joint name="Revolute 2" type="continuous">
+  <joint name="Revolute2" type="continuous">
     <origin xyz="0.5 0.0 0.25" rpy="0 0 0"/>
-    <parent link="base_link"/>
+    <parent link="chassis"/>
     <child link="right_wheel_1"/>
     <axis xyz="1.0 0.0 0.0"/>
   </joint>
+  <gazebo reference="left_wheel_1">
+    <mu1 value="0.001"/>
+    <mu2 value="0.001"/>
+  </gazebo>
+  <gazebo reference="right_wheel_1">
+    <mu1 value="0.001"/>
+    <mu2 value="0.001"/>
+  </gazebo>
 </robot>

File: src/basic_robot/description/test.xacro (robot description, xacro)
@@ -1,7 +1,7 @@
 <?xml version="1.0" ?>
-<robot name="test" xmlns:xacro="http://www.ros.org/wiki/xacro">
+<robot name="Basic_Robot" xmlns:xacro="http://www.ros.org/wiki/xacro">
   <link name="base_link">
   </link>
-  <joint name="base_joint" type="fixed">
+  <joint name="base_chassis_joint" type="fixed">
     <parent link="base_link"/>
     <child link="chassis"/>
@@ -11,35 +11,7 @@
       <origin xyz="0 0 0" rpy="0 0 0"/>
       <geometry>
-        <mesh filename="package://basic_robot/meshes/chassis.stl" scale="0.1 0.1 0.1"/>
+        <mesh filename="package://basic_robot/meshes/left_wheel_1.stl" scale="0.01 0.01 0.01"/>
       </geometry>
     </visual>
   </link>
-  <link name="left_wheel_1">
-    <visual>
-      <origin xyz="0.5 -0.0 -0.25" rpy="0 0 0"/>
-      <geometry>
-        <mesh filename="package://basic_robot/meshes/left_wheel_1.stl" scale="0.1 0.1 0.1"/>
-      </geometry>
-    </visual>
-  </link>
-  <link name="right_wheel_1">
-    <visual>
-      <origin xyz="-0.5 -0.0 -0.25" rpy="0 0 0"/>
-      <geometry>
-        <mesh filename="package://basic_robot/meshes/right_wheel_1.stl" scale="0.1 0.1 0.1"/>
-      </geometry>
-    </visual>
-  </link>
-  <joint name="Revolute 1" type="continuous">
-    <origin xyz="-0.5 0.0 0.25" rpy="0 0 0"/>
-    <parent link="chassis"/>
-    <child link="left_wheel_1"/>
-    <axis xyz="-1.0 0.0 0.0"/>
-  </joint>
-  <joint name="Revolute 2" type="continuous">
-    <origin xyz="0.5 0.0 0.25" rpy="0 0 0"/>
-    <parent link="chassis"/>
-    <child link="right_wheel_1"/>
-    <axis xyz="1.0 0.0 0.0"/>
-  </joint>
 </robot>
