Commit message: ros2_control still isn't working

File: src/basic_robot/description/main.xacro (robot description, xacro)
@@ -2,4 +2,37 @@
 <robot name="my_bot" xmlns:xacro="http://www.ros.org/wiki/xacro">
     <xacro:include filename="gazebo.xacro"/>
-    <xacro:include filename="ros2_control.xacro"/>
+    <gazebo reference="chassis">
+        <material>
+            Gazebo/Green
+        </material>
+    </gazebo>
+    <ros2_control name="GazeboSystem" type="system">
+        <hardware>
+            <plugin>
+                gazebo_ros2_control/GazeboSystem
+            </plugin>
+        </hardware>
+        <joint name="Revolute1">
+            <command_interface name="velocity">
+                <param name="min">-10</param>
+                <param name="max">10</param>
+            </command_interface>
+            <state_interface name="velocity"/>
+            <state_interface name="position"/>
+        </joint>
+        <joint name="Revolute2">
+            <command_interface name="velocity">
+                <param name="min">-10</param>
+                <param name="max">10</param>
+            </command_interface>
+            <state_interface name="velocity"/>
+            <state_interface name="position"/>
+        </joint>
+    </ros2_control>
+    <gazebo>
+        <plugin filename="libgazebo_ros2_control.so" name="gazebo_ros2_control" >
+            <parameters>$(find basic_robot)/config/my_controllers.yaml</parameters>
+        </plugin>
+    </gazebo>
+    <!--<xacro:include filename="ros2_control.xacro"/>-->
 </robot>

File: src/basic_robot/description/ros2_control.xacro (robot description, xacro)
@@ -25,5 +25,5 @@
     </ros2_control>
     <gazebo>
-        <plugin name="gazebo_ros2_control" filename="libgazebo_ros2_control.so">
+        <plugin filename="libgazebo_ros2_control.so" name="gazebo_ros2_control" >
             <parameters>$(find basic_robot)/config/my_controllers.yaml</parameters>
         </plugin>
